File: s1_ipod_serial.sch (KiCad schematic (older format))
At the start: 32 parts, among them IC1 GL850G-LQFP48, J1 USB-MINIB-5PIN, P1 IPOD_CONNECTOR_MALE, U1 LM3526M-H, U2 FT232RL-BASICSSOP, X1 12 Mhz

Commit message: new routing for usb, teileliste added, fix for selfpowered
Parts:
- added D1: Suspend, symbol LED
- added R3, R4, R7, R8: 0R, symbol R
Connections:
- net DVDD: now also D1.1 (A), R3.1
- net GND: now also P1.1 (GND@1), R5.1, R4.1; no longer IC1.37 (PSELF)
- net IPOD_USB_D+: now also R8.2; no longer P1.27 (USB_D+)
- net IPOD_USB_D-: now also R7.2; no longer P1.25 (USB_D-)
- net at IC1.39 (PGANG), R6.1: now also D1.2 (K)
- new net: P1.25 (USB_D-), R7.1
- new net: P1.27 (USB_D+), R8.1
- new net: IC1.37 (PSELF), R3.2, R4.2

Commit message: added some teile
Parts:
- R1: value 480R -> 470R
Changed lines of the file:
@@
 P 2900 2850
 F 0 "R1" V 2980 2850 40  0000 C CNN
-F 1 "480R" V 2907 2851 40  0000 C CNN
+F 1 "470R" V 2907 2851 40  0000 C CNN
 F 2 "" V 2830 2850 30  0000 C CNN
 F 3 "" H 2900 2850 30  0000 C CNN

Commit message: removed the 0R for self powered indicator, made fb 0608, rev. text added to board and sheet, routing optimized
Parts:
- removed R3, R4: 0R, symbol R
Connections:
- net DVDD: now also IC1.37 (PSELF)
- no-connect marks 38 -> 41
Changed lines of the file:
@@
 encoding utf-8
 Sheet 1 1
-Title "iPod Serialcable"
-Date "25 Mär 2014"
-Rev "0.9"
+Title "iPod Serial Connector"
+Date "06 Jun 2014"
+Rev "0.8"
 Comp "SektionEins GmbH"
 Comment1 ""
@@
 	1    0    0    -1
 $EndComp
-$Comp
-L R R3
-U 1 1 538C963C
-P 4050 2750
-F 0 "R3" V 4130 2750 40  0000 C CNN
-F 1 "0R" V 4057 2751 40  0000 C CNN
-F 2 "" V 3980 2750 30  0000 C CNN
-F 3 "" H 4050 2750 30  0000 C CNN
-	1    4050 2750
-	1    0    0    -1
-$EndComp
-$Comp
-L R R4
-U 1 1 538C9650
-P 4200 2750
-F 0 "R4" V 4280 2750 40  0000 C CNN
-F 1 "0R" V 4207 2751 40  0000 C CNN
-F 2 "" V 4130 2750 30  0000 C CNN
-F 3 "" H 4200 2750 30  0000 C CNN
-	1    4200 2750
-	1    0    0    -1
-$EndComp
 Wire Wire Line
 	8850 2200 9700 2200
@@
 	5250 4550 5250 4600
 Wire Wire Line
-	4550 4600 6900 4600
+	6900 4600 4550 4600
 Wire Wire Line
 	5850 4600 5850 4550
@@
 	6150 4750 6150 4550
 Wire Wire Line
-	4050 2450 6250 2450
-Wire Wire Line
 	5350 2450 5350 2550
 Wire Wire Line
@@
 	4500 4100 4600 4100
 Connection ~ 4500 3700
-Connection ~ 4500 2450
-Wire Wire Line
-	4550 2500 4550 4600
+Wire Wire Line
+	4550 4600 4550 2500
 Connection ~ 5250 4600
 Wire Wire Line
@@
 Wire Wire Line
 	4450 4000 4600 4000
-Wire Wire Line
-	4200 2500 6050 2500
 Wire Wire Line
 	6050 2500 6050 2550
@@
 	9350 800  9350 700
 Connection ~ 9550 700
-Wire Wire Line
-	4050 3000 4600 3000
-Connection ~ 4200 3000
-Connection ~ 4550 2500
-Wire Wire Line
-	4050 2450 4050 2500
 $Comp
 L LED D1
@@
 	0    1    1    0
 $EndComp
+Wire Wire Line
+	4550 2500 6050 2500
+Wire Wire Line
+	4600 3000 4500 3000
+Connection ~ 4500 3000
+Wire Wire Line
+	4500 2450 6250 2450
+Connection ~ 4500 2450
+NoConn ~ 2650 3900
+NoConn ~ 1950 3900
+NoConn ~ 1950 3800
 $EndSCHEMATC

Commit message: added current version
Parts:
- C5: value 0,1uF -> 100nF
- U1: value LM3526M-H -> LM3526M-L
Connections:
- net DVDD: no longer IC1.33 (PAMDER3), IC1.36 (PAMBER2), IC1.45 (PGREEN1)
- net GND: no longer IC1.24 (PAMBER4)
- no-connect marks 41 -> 45
Changed lines of the file:
@@
 Sheet 1 1
 Title "iPod Serial Connector"
-Date "06 Jun 2014"
-Rev "0.8"
+Date "07 Jul 2014"
+Rev "0.5"
 Comp "SektionEins GmbH"
 Comment1 ""
@@
 P 9350 2550
 F 0 "C5" H 9350 2650 40  0000 L CNN
-F 1 "0,1uF" H 9356 2465 40  0000 L CNN
+F 1 "100nF" H 9356 2465 40  0000 L CNN
 F 2 "" H 9388 2400 30  0000 C CNN
 F 3 "" H 9350 2550 60  0000 C CNN
@@
 P 2350 3700
 F 0 "U1" H 2300 3950 50  0000 C CNN
-F 1 "LM3526M-H" H 2300 3350 50  0000 C CNN
+F 1 "LM3526M-L" H 2300 3350 50  0000 C CNN
 F 2 "" H 2350 3700 60  0000 C CNN
 F 3 "" H 2350 3700 60  0000 C CNN
@@
 	5850 4600 5850 4550
 Wire Wire Line
-	6900 3000 6900 4750
-Wire Wire Line
 	6900 4100 6850 4100
 Connection ~ 5850 4600
@@
 Connection ~ 7750 4250
 Wire Wire Line
-	5150 2550 5150 2450
-Connection ~ 5150 2450
-Wire Wire Line
-	6850 3000 6900 3000
-Connection ~ 6900 3400
-Wire Wire Line
-	5450 2550 5450 2450
-Connection ~ 5450 2450
-Wire Wire Line
 	2550 2850 2650 2850
 Wire Wire Line
 	6850 3500 6950 3500
 Connection ~ 6950 3500
-Wire Wire Line
-	4600 3800 4500 3800
-Connection ~ 4500 3800
 Wire Wire Line
 	9350 800  9350 700
@@
 NoConn ~ 1950 3900
 NoConn ~ 1950 3800
+NoConn ~ 4600 3800
+NoConn ~ 5150 2550
+NoConn ~ 5450 2550
+NoConn ~ 6850 3000
+Wire Wire Line
+	6900 3400 6900 4750
 $EndSCHEMATC
